File: Kicad Files/Remote/Cable Test Remote.sch (KiCad schematic (older format))
At the start: 20 parts, among them J1 RJ45, J2 RJ12

Commit message: Begin PCB layout
Parts:
- D1, D2, D3, D4, D5, D6, D7, D8, D9: footprint (none) -> Diodes_SMD:SOD-123
- J1: footprint (none) -> Tester_Connectors:RJ45_SHLD
- J2: footprint (none) -> Tester_Connectors:RJ12_SHLD
- LED1, LED2, LED3, LED4, LED5, LED6, LED7, LED8, LED9: footprint (none) -> LEDs:LED-3MM
Changed lines of the file:
@@
 F 0 "J2" H 6100 3150 50  0000 C CNN
 F 1 "RJ12" H 5750 3150 50  0000 C CNN
-F 2 "" H 5900 2650 50  0000 C CNN
+F 2 "Tester_Connectors:RJ12_SHLD" H 5900 2650 50  0001 C CNN
 F 3 "" H 5900 2650 50  0000 C CNN
 	1    5900 2650
@@
 F 0 "J1" H 4950 3150 50  0000 C CNN
 F 1 "RJ45" H 4600 3150 50  0000 C CNN
-F 2 "" H 4750 2650 50  0000 C CNN
+F 2 "Tester_Connectors:RJ45_SHLD" H 4750 2650 50  0001 C CNN
 F 3 "" H 4750 2650 50  0000 C CNN
 	1    4750 2650
@@
 F 0 "LED1" H 2800 1400 50  0000 C CNN
 F 1 "LED" H 2800 1200 50  0000 C CNN
-F 2 "" H 2800 1300 50  0000 C CNN
+F 2 "LEDs:LED-3MM" H 2800 1300 50  0001 C CNN
 F 3 "" H 2800 1300 50  0000 C CNN
 	1    2800 1300
@@
 F 0 "D1" H 2750 1700 50  0000 C CNN
 F 1 "D" H 2750 1500 50  0000 C CNN
-F 2 "" H 2750 1600 50  0000 C CNN
+F 2 "Diodes_SMD:SOD-123" H 2750 1600 50  0001 C CNN
 F 3 "" H 2750 1600 50  0000 C CNN
 	1    2750 1600
@@
 F 0 "LED2" H 2800 2000 50  0000 C CNN
 F 1 "LED" H 2800 1800 50  0000 C CNN
-F 2 "" H 2800 1900 50  0000 C CNN
+F 2 "LEDs:LED-3MM" H 2800 1900 50  0001 C CNN
 F 3 "" H 2800 1900 50  0000 C CNN
 	1    2800 1900
@@
 F 0 "D2" H 2750 2300 50  0000 C CNN
 F 1 "D" H 2750 2100 50  0000 C CNN
-F 2 "" H 2750 2200 50  0000 C CNN
+F 2 "Diodes_SMD:SOD-123" H 2750 2200 50  0001 C CNN
 F 3 "" H 2750 2200 50  0000 C CNN
 	1    2750 2200
@@
 F 0 "LED3" H 2800 2600 50  0000 C CNN
 F 1 "LED" H 2800 2400 50  0000 C CNN
-F 2 "" H 2800 2500 50  0000 C CNN
+F 2 "LEDs:LED-3MM" H 2800 2500 50  0001 C CNN
 F 3 "" H 2800 2500 50  0000 C CNN
 	1    2800 2500
@@
 F 0 "D3" H 2750 2900 50  0000 C CNN
 F 1 "D" H 2750 2700 50  0000 C CNN
-F 2 "" H 2750 2800 50  0000 C CNN
+F 2 "Diodes_SMD:SOD-123" H 2750 2800 50  0001 C CNN
 F 3 "" H 2750 2800 50  0000 C CNN
 	1    2750 2800
@@
 F 0 "LED4" H 2800 3200 50  0000 C CNN
 F 1 "LED" H 2800 3000 50  0000 C CNN
-F 2 "" H 2800 3100 50  0000 C CNN
+F 2 "LEDs:LED-3MM" H 2800 3100 50  0001 C CNN
 F 3 "" H 2800 3100 50  0000 C CNN
 	1    2800 3100
@@
 F 0 "D4" H 2750 3500 50  0000 C CNN
 F 1 "D" H 2750 3300 50  0000 C CNN
-F 2 "" H 2750 3400 50  0000 C CNN
+F 2 "Diodes_SMD:SOD-123" H 2750 3400 50  0001 C CNN
 F 3 "" H 2750 3400 50  0000 C CNN
 	1    2750 3400
@@
 F 0 "LED5" H 2800 3800 50  0000 C CNN
 F 1 "LED" H 2800 3600 50  0000 C CNN
-F 2 "" H 2800 3700 50  0000 C CNN
+F 2 "LEDs:LED-3MM" H 2800 3700 50  0001 C CNN
 F 3 "" H 2800 3700 50  0000 C CNN
 	1    2800 3700
@@
 F 0 "D5" H 2750 4100 50  0000 C CNN
 F 1 "D" H 2750 3900 50  0000 C CNN
-F 2 "" H 2750 4000 50  0000 C CNN
+F 2 "Diodes_SMD:SOD-123" H 2750 4000 50  0001 C CNN
 F 3 "" H 2750 4000 50  0000 C CNN
 	1    2750 4000
@@
 F 0 "LED6" H 2800 4400 50  0000 C CNN
 F 1 "LED" H 2800 4200 50  0000 C CNN
-F 2 "" H 2800 4300 50  0000 C CNN
+F 2 "LEDs:LED-3MM" H 2800 4300 50  0001 C CNN
 F 3 "" H 2800 4300 50  0000 C CNN
 	1    2800 4300
@@
 F 0 "D6" H 2750 4700 50  0000 C CNN
 F 1 "D" H 2750 4500 50  0000 C CNN
-F 2 "" H 2750 4600 50  0000 C CNN
+F 2 "Diodes_SMD:SOD-123" H 2750 4600 50  0001 C CNN
 F 3 "" H 2750 4600 50  0000 C CNN
 	1    2750 4600
@@
 F 0 "LED7" H 2800 5000 50  0000 C CNN
 F 1 "LED" H 2800 4800 50  0000 C CNN
-F 2 "" H 2800 4900 50  0000 C CNN
+F 2 "LEDs:LED-3MM" H 2800 4900 50  0001 C CNN
 F 3 "" H 2800 4900 50  0000 C CNN
 	1    2800 4900
@@
 F 0 "D7" H 2750 5300 50  0000 C CNN
 F 1 "D" H 2750 5100 50  0000 C CNN
-F 2 "" H 2750 5200 50  0000 C CNN
+F 2 "Diodes_SMD:SOD-123" H 2750 5200 50  0001 C CNN
 F 3 "" H 2750 5200 50  0000 C CNN
 	1    2750 5200
@@
 F 0 "LED8" H 2800 5600 50  0000 C CNN
 F 1 "LED" H 2800 5400 50  0000 C CNN
-F 2 "" H 2800 5500 50  0000 C CNN
+F 2 "LEDs:LED-3MM" H 2800 5500 50  0001 C CNN
 F 3 "" H 2800 5500 50  0000 C CNN
 	1    2800 5500
@@
 F 0 "D8" H 2750 5900 50  0000 C CNN
 F 1 "D" H 2750 5700 50  0000 C CNN
-F 2 "" H 2750 5800 50  0000 C CNN
+F 2 "Diodes_SMD:SOD-123" H 2750 5800 50  0001 C CNN
 F 3 "" H 2750 5800 50  0000 C CNN
 	1    2750 5800
@@
 F 0 "LED9" H 2800 6200 50  0000 C CNN
 F 1 "LED" H 2800 6000 50  0000 C CNN
-F 2 "" H 2800 6100 50  0000 C CNN
+F 2 "LEDs:LED-3MM" H 2800 6100 50  0001 C CNN
 F 3 "" H 2800 6100 50  0000 C CNN
 	1    2800 6100
@@
 F 0 "D9" H 2750 6500 50  0000 C CNN
 F 1 "D" H 2750 6300 50  0000 C CNN
-F 2 "" H 2750 6400 50  0000 C CNN
+F 2 "Diodes_SMD:SOD-123" H 2750 6400 50  0001 C CNN
 F 3 "" H 2750 6400 50  0000 C CNN
 	1    2750 6400
