File: Kicad Files/Remote/Cable Test Remote.kicad_pcb (KiCad board)
At the start: 2 copper layers, 25.4 x 96.5 mm, 23 parts, among them J1 RJ45, J2 RJ12

Commit message: Shorten Remote board to better fit case
Parts:
- moved J2 0.64 mm to (114.3, 141.6)
Routing:
- net /S: track 159.1 -> 158.5 mm
- net /3: track 140.3 -> 139.7 mm
- net /6: track 150.7 -> 150.1 mm
- net /5: track 145.4 -> 144.8 mm
- net /4: track 145.9 -> 145.3 mm
- net /2: track 131.0 -> 130.4 mm
- net /1: track 116.4 -> 115.8 mm
Other:
- board size 25.4 x 96.5 mm -> 25.4 x 95.9 mm
- board text added: "Cable Tester Remote v0.2"
- board text removed: "Cable Tester Remote v0.1"
