File: Kicad Files/Master/Cable Test Master.sch (KiCad schematic (older format))
At the start: 32 parts, among them J1 RJ45, J2 RJ12, J3 PWR, J4 ISP, SW2 DP3T, U1 ATTINY24-SS, U2 78L05

Commit message: Change R1-R9 to 100 ohm
Changed lines of the file:
@@
 Title "Cable Tester, Master End"
 Date "2018-01-06"
-Rev "0.2"
+Rev "0.3"
 Comp ""
 Comment1 ""
@@
 	3600 3700 3800 3700
 Wire Wire Line
-	3800 4850 3800 3700
-Wire Wire Line
-	2300 4850 3800 4850
+	3800 3700 3800 4850
+Wire Wire Line
+	3800 4850 2300 4850
 Wire Wire Line
 	3000 4850 3000 4700
@@
 D2
 Wire Bus Line
-	7200 5300 6200 5300
+	6200 5300 7200 5300
 Entry Wire Line
 	7200 2700 7300 2600
@@
 	7200 3300 7300 3200
 Wire Bus Line
-	7200 2700 7200 5300
+	7200 5300 7200 2700
 Wire Wire Line
 	7300 3200 7400 3200

Commit message: Change SW2 reference to SW1
Parts:
- renumbered SW2 to SW1
Changed lines of the file:
@@
 $EndSheet
 $Comp
-L DP3T SW2
+L DP3T SW1
 U 1 1 5A59345F
 P 1850 4700
-F 0 "SW2" H 1850 4300 60  0000 C CNN
+F 0 "SW1" H 1850 4300 60  0000 C CNN
 F 1 "DP3T" H 1850 5100 60  0000 C CNN
 F 2 "Tester Switches:SW_DP3T_SLIDE" H 1800 4600 60  0001 C CNN
