File: Kicad Files/Master/MOSFET Drive.sch (KiCad schematic (older format))
At the start: 27 parts, among them Q1 BSS84, Q10 2N7002, Q11 2N7002, Q12 2N7002, Q13 2N7002, Q14 2N7002, Q15 2N7002, Q16 2N7002, Q17 2N7002, Q18 2N7002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

Commit message: Fix P-channel MOSFET wiring and software output levels
Connections:
- net DRIVE_1: now also Q1.3 (D); no longer Q1.2 (S)
- net DRIVE_2: now also Q2.3 (D); no longer Q2.2 (S)
- net DRIVE_3: now also Q3.3 (D); no longer Q3.2 (S)
- net DRIVE_4: now also Q4.3 (D); no longer Q4.2 (S)
- net DRIVE_5: now also Q5.3 (D); no longer Q5.2 (S)
- net DRIVE_6: now also Q6.3 (D); no longer Q6.2 (S)
- net DRIVE_7: now also Q7.3 (D); no longer Q7.2 (S)
- net DRIVE_8: now also Q8.3 (D); no longer Q8.2 (S)
- net DRIVE_S: now also Q9.3 (D); no longer Q9.2 (S)
- net at R1.2: now also Q1.2 (S); no longer Q1.3 (D)
- net at R2.2: now also Q2.2 (S); no longer Q2.3 (D)
- net at R3.2: now also Q3.2 (S); no longer Q3.3 (D)
- net at R4.2: now also Q4.2 (S); no longer Q4.3 (D)
- net at R5.2: now also Q5.2 (S); no longer Q5.3 (D)
- net at R6.2: now also Q6.2 (S); no longer Q6.3 (D)
- net at R7.2: now also Q7.2 (S); no longer Q7.3 (D)
- net at R8.2: now also Q8.2 (S); no longer Q8.3 (D)
- net at R9.2: now also Q9.2 (S); no longer Q9.3 (D)
Changed lines of the file:
@@
 F 3 "" H 8500 2300 50  0000 C CNN
 	1    8500 2300
-	1    0    0    -1
+	1    0    0    1
 $EndComp
 $Comp
@@
 F 3 "" H 7700 2300 50  0000 C CNN
 	1    7700 2300
-	1    0    0    -1
+	1    0    0    1
 $EndComp
 $Comp
@@
 F 3 "" H 6900 2300 50  0000 C CNN
 	1    6900 2300
-	1    0    0    -1
+	1    0    0    1
 $EndComp
 $Comp
@@
 F 3 "" H 6100 2300 50  0000 C CNN
 	1    6100 2300
-	1    0    0    -1
+	1    0    0    1
 $EndComp
 $Comp
@@
 F 3 "" H 5300 2300 50  0000 C CNN
 	1    5300 2300
-	1    0    0    -1
+	1    0    0    1
 $EndComp
 $Comp
@@
 F 3 "" H 4500 2300 50  0000 C CNN
 	1    4500 2300
-	1    0    0    -1
+	1    0    0    1
 $EndComp
 $Comp
@@
 F 3 "" H 3700 2300 50  0000 C CNN
 	1    3700 2300
-	1    0    0    -1
+	1    0    0    1
 $EndComp
 $Comp
@@
 F 3 "" H 2900 2300 50  0000 C CNN
 	1    2900 2300
-	1    0    0    -1
+	1    0    0    1
 $EndComp
 $Comp
@@
 F 3 "" H 2100 2300 50  0000 C CNN
 	1    2100 2300
-	1    0    0    -1
+	1    0    0    1
 $EndComp
 $EndSCHEMATC

Commit message: Change R1-R9 to 100 ohm
Parts:
- R1, R2, R3, R4, R5, R6, R7, R8, R9: value 160 -> 100
Changed lines of the file:
@@
 P 2200 1650
 F 0 "R1" V 2280 1650 50  0000 C CNN
-F 1 "160" V 2200 1650 50  0000 C CNN
+F 1 "100" V 2200 1650 50  0000 C CNN
 F 2 "Resistors_SMD:R_0805_HandSoldering" V 2130 1650 50  0001 C CNN
 F 3 "" H 2200 1650 50  0000 C CNN
@@
 P 3000 1650
 F 0 "R2" V 3080 1650 50  0000 C CNN
-F 1 "160" V 3000 1650 50  0000 C CNN
+F 1 "100" V 3000 1650 50  0000 C CNN
 F 2 "Resistors_SMD:R_0805_HandSoldering" V 2930 1650 50  0001 C CNN
 F 3 "" H 3000 1650 50  0000 C CNN
@@
 P 3800 1650
 F 0 "R3" V 3880 1650 50  0000 C CNN
-F 1 "160" V 3800 1650 50  0000 C CNN
+F 1 "100" V 3800 1650 50  0000 C CNN
 F 2 "Resistors_SMD:R_0805_HandSoldering" V 3730 1650 50  0001 C CNN
 F 3 "" H 3800 1650 50  0000 C CNN
@@
 P 4600 1650
 F 0 "R4" V 4680 1650 50  0000 C CNN
-F 1 "160" V 4600 1650 50  0000 C CNN
+F 1 "100" V 4600 1650 50  0000 C CNN
 F 2 "Resistors_SMD:R_0805_HandSoldering" V 4530 1650 50  0001 C CNN
 F 3 "" H 4600 1650 50  0000 C CNN
@@
 P 5400 1650
 F 0 "R5" V 5480 1650 50  0000 C CNN
-F 1 "160" V 5400 1650 50  0000 C CNN
+F 1 "100" V 5400 1650 50  0000 C CNN
 F 2 "Resistors_SMD:R_0805_HandSoldering" V 5330 1650 50  0001 C CNN
 F 3 "" H 5400 1650 50  0000 C CNN
@@
 P 6200 1650
 F 0 "R6" V 6280 1650 50  0000 C CNN
-F 1 "160" V 6200 1650 50  0000 C CNN
+F 1 "100" V 6200 1650 50  0000 C CNN
 F 2 "Resistors_SMD:R_0805_HandSoldering" V 6130 1650 50  0001 C CNN
 F 3 "" H 6200 1650 50  0000 C CNN
@@
 P 7000 1650
 F 0 "R7" V 7080 1650 50  0000 C CNN
-F 1 "160" V 7000 1650 50  0000 C CNN
+F 1 "100" V 7000 1650 50  0000 C CNN
 F 2 "Resistors_SMD:R_0805_HandSoldering" V 6930 1650 50  0001 C CNN
 F 3 "" H 7000 1650 50  0000 C CNN
@@
 P 7800 1650
 F 0 "R8" V 7880 1650 50  0000 C CNN
-F 1 "160" V 7800 1650 50  0000 C CNN
+F 1 "100" V 7800 1650 50  0000 C CNN
 F 2 "Resistors_SMD:R_0805_HandSoldering" V 7730 1650 50  0001 C CNN
 F 3 "" H 7800 1650 50  0000 C CNN
@@
 P 8600 1650
 F 0 "R9" V 8680 1650 50  0000 C CNN
-F 1 "160" V 8600 1650 50  0000 C CNN
+F 1 "100" V 8600 1650 50  0000 C CNN
 F 2 "Resistors_SMD:R_0805_HandSoldering" V 8530 1650 50  0001 C CNN
 F 3 "" H 8600 1650 50  0000 C CNN

Commit message: Change current limiting resistors to 200 Ohm
The 100 Ohm resistors worked but the LEDs burn rather bright. Increasing resistance to be easier on eyes. Also changed BOM to match.
Parts:
- R1, R2, R3, R4, R5, R6, R7, R8, R9: value 100 -> 200
Changed lines of the file:
@@
 P 2200 1650
 F 0 "R1" V 2280 1650 50  0000 C CNN
-F 1 "100" V 2200 1650 50  0000 C CNN
+F 1 "200" V 2200 1650 50  0000 C CNN
 F 2 "Resistors_SMD:R_0805_HandSoldering" V 2130 1650 50  0001 C CNN
 F 3 "" H 2200 1650 50  0000 C CNN
@@
 P 3000 1650
 F 0 "R2" V 3080 1650 50  0000 C CNN
-F 1 "100" V 3000 1650 50  0000 C CNN
+F 1 "200" V 3000 1650 50  0000 C CNN
 F 2 "Resistors_SMD:R_0805_HandSoldering" V 2930 1650 50  0001 C CNN
 F 3 "" H 3000 1650 50  0000 C CNN
@@
 P 3800 1650
 F 0 "R3" V 3880 1650 50  0000 C CNN
-F 1 "100" V 3800 1650 50  0000 C CNN
+F 1 "200" V 3800 1650 50  0000 C CNN
 F 2 "Resistors_SMD:R_0805_HandSoldering" V 3730 1650 50  0001 C CNN
 F 3 "" H 3800 1650 50  0000 C CNN
@@
 P 4600 1650
 F 0 "R4" V 4680 1650 50  0000 C CNN
-F 1 "100" V 4600 1650 50  0000 C CNN
+F 1 "200" V 4600 1650 50  0000 C CNN
 F 2 "Resistors_SMD:R_0805_HandSoldering" V 4530 1650 50  0001 C CNN
 F 3 "" H 4600 1650 50  0000 C CNN
@@
 P 5400 1650
 F 0 "R5" V 5480 1650 50  0000 C CNN
-F 1 "100" V 5400 1650 50  0000 C CNN
+F 1 "200" V 5400 1650 50  0000 C CNN
 F 2 "Resistors_SMD:R_0805_HandSoldering" V 5330 1650 50  0001 C CNN
 F 3 "" H 5400 1650 50  0000 C CNN
@@
 P 6200 1650
 F 0 "R6" V 6280 1650 50  0000 C CNN
-F 1 "100" V 6200 1650 50  0000 C CNN
+F 1 "200" V 6200 1650 50  0000 C CNN
 F 2 "Resistors_SMD:R_0805_HandSoldering" V 6130 1650 50  0001 C CNN
 F 3 "" H 6200 1650 50  0000 C CNN
@@
 P 7000 1650
 F 0 "R7" V 7080 1650 50  0000 C CNN
-F 1 "100" V 7000 1650 50  0000 C CNN
+F 1 "200" V 7000 1650 50  0000 C CNN
 F 2 "Resistors_SMD:R_0805_HandSoldering" V 6930 1650 50  0001 C CNN
 F 3 "" H 7000 1650 50  0000 C CNN
@@
 P 7800 1650
 F 0 "R8" V 7880 1650 50  0000 C CNN
-F 1 "100" V 7800 1650 50  0000 C CNN
+F 1 "200" V 7800 1650 50  0000 C CNN
 F 2 "Resistors_SMD:R_0805_HandSoldering" V 7730 1650 50  0001 C CNN
 F 3 "" H 7800 1650 50  0000 C CNN
@@
 P 8600 1650
 F 0 "R9" V 8680 1650 50  0000 C CNN
-F 1 "100" V 8600 1650 50  0000 C CNN
+F 1 "200" V 8600 1650 50  0000 C CNN
 F 2 "Resistors_SMD:R_0805_HandSoldering" V 8530 1650 50  0001 C CNN
 F 3 "" H 8600 1650 50  0000 C CNN
